Commit message: Port mir gazebo simulation to ros2 jazzy and Gazebo harmonic

File: mir_description/urdf/include/common_properties.urdf.xacro (robot description, xacro)
@@ -3,5 +3,5 @@
   Various useful properties such as constants and materials
  -->
-<robot name="xacro_properties" xmlns:xacro="http://ros.org/wiki/xacro">
+<robot name="xacro_properties" xmlns:xacro="http://www.ros.org/wiki/xacro">
   <!-- #################### RViz materials #################### -->
   <xacro:property name="material_white">

File: mir_description/urdf/include/mir.gazebo.xacro (robot description, xacro)
@@ -1,35 +1,69 @@
 <?xml version="1.0"?>
-<robot xmlns:xacro="http://ros.org/wiki/xacro">
-  <!-- See https://github.com/ros-simulation/gazebo_ros_pkgs/wiki/ROS-2-Migration:-Diff-drive for ros2 information -->
-  <xacro:macro name="diff_controller_plugin_gazebo" params="prefix ns left_wheel_joint right_wheel_joint wheel_separation wheel_radius">
+<robot xmlns:xacro="http://www.ros.org/wiki/xacro">
+  <xacro:macro name="sensors_system_plugin" params="">
     <gazebo>
-      <!-- Use gazebo_ros_joint_state_publisher instead of publishWheelJointState -->
-      <plugin name="joint_states" filename="libgazebo_ros_joint_state_publisher.so">
-        <ros>
-          <namespace>${ns}</namespace>
-        </ros>
-        <update_rate>1000.0</update_rate>
-        <joint_name>${right_wheel_joint}</joint_name>
-        <joint_name>${left_wheel_joint}</joint_name>
+      <!-- Required by lidar in simulation -->
+      <plugin filename="gz-sim-sensors-system" name="gz::sim::systems::Sensors"/>
+    </gazebo>
+  </xacro:macro>
+  <!-- plugin to publish joint states, see code under
+         https://github.com/gazebosim/gz-sim/blob/gz-sim8/src/systems/joint_state_publisher/JointStatePublisher.hh -->
+  <xacro:macro name="joint_states_plugin_gazebo" params="prefix topic left_wheel_joint right_wheel_joint">
+    <gazebo>
+      <plugin filename="gz-sim-joint-state-publisher-system" name="gz::sim::systems::JointStatePublisher">
+        <topic>${prefix}${topic}</topic>
+        <joint_name>${prefix}${left_wheel_joint}</joint_name>
+        <joint_name>${prefix}${right_wheel_joint}</joint_name>
+        <!-- publishing the caster wheels joints is possible in simulation uncommenting this sections of the code
+             but the real robot does not has enconders in the caster wheels.
+             Furthermore it helps to save bandwidth not to publish them.
+        <joint_name>${prefix}fl_caster_wheel_joint</joint_name>
+        <joint_name>${prefix}fr_caster_wheel_joint</joint_name>
+        <joint_name>${prefix}bl_caster_wheel_joint</joint_name>
+        <joint_name>${prefix}br_caster_wheel_joint</joint_name>
+        <joint_name>${prefix}fl_caster_rotation_joint</joint_name>
+        <joint_name>${prefix}fr_caster_rotation_joint</joint_name>
+        <joint_name>${prefix}bl_caster_rotation_joint</joint_name>
+        <joint_name>${prefix}br_caster_rotation_joint</joint_name> -->
       </plugin>
-      <plugin name="diff_drive_controller" filename="libgazebo_ros_diff_drive.so">
-        <ros>
-          <remapping>cmd_vel:=${prefix}cmd_vel</remapping>
-          <remapping>odom:=${prefix}odom</remapping>
-        </ros>
-        <legacy_mode>false</legacy_mode>
-        <always_on>true</always_on>
-        <update_rate>1000.0</update_rate>
+    </gazebo>
+  </xacro:macro>
+  <!-- diff drive plugin, see code under
+         https://github.com/gazebosim/gz-sim/blob/gz-sim8/src/systems/diff_drive/DiffDrive.hh -->
+  <xacro:macro name="diff_controller_plugin_gazebo" params="prefix left_wheel_joint right_wheel_joint wheel_separation wheel_radius">
+    <gazebo>
+      <plugin filename="gz-sim-diff-drive-system" name="gz::sim::systems::DiffDrive">
+        <!-- wheels -->
         <left_joint>${left_wheel_joint}</left_joint>
         <right_joint>${right_wheel_joint}</right_joint>
+        <!-- kinematics -->
         <wheel_separation>${wheel_separation}</wheel_separation>
-        <wheel_diameter>${2*wheel_radius}</wheel_diameter>
-        <odometry_frame>${prefix}odom</odometry_frame>
-        <robot_base_frame>${prefix}base_footprint</robot_base_frame>
-        <publish_odom>true</publish_odom>
-        <publish_wheel_tf>false</publish_wheel_tf>
-        <publish_odom_tf>true</publish_odom_tf>
-        <max_wheel_torque>10</max_wheel_torque>
-        <max_wheel_acceleration>2.8</max_wheel_acceleration>
+        <wheel_radius>${wheel_radius}</wheel_radius>
+        <!-- limits
+          The following params could be set if needed
+          min_velocity - Sets both the minimum linear and minimum angular velocity.
+          min_linear_velocity - Sets the minimum linear velocity. Overrides `<min_velocity>` if set.
+          min_angular_velocity - Sets the minimum angular velocity. Overrides `<min_velocity>` if set.
+          max_velocity - Sets both the maximum linear and maximum angular velocity.
+          max_linear_velocity - Sets the maximum linear velocity. Overrides `<max_velocity>` if set.
+          max_angular_velocity - Sets the maximum angular velocity. Overrides `<max_velocity>` if set.
+          min_acceleration - Sets both the minimum linear and minimum angular acceleration.
+          min_linear_acceleration - Sets the minimum linear acceleration. Overrides `<min_acceleration>` if set.
+          min_angular_acceleration - Sets the minimum angular acceleration. Overrides `<min_acceleration>` if set.
+          max_acceleration - Sets both the maximum linear and maximum angular acceleration.
+        -->
+        <max_linear_acceleration>2.8</max_linear_acceleration>
+        <!-- max_angular_acceleration (could be set if needed) - Sets the maximum angular acceleration.
+                                                                 Overrides `<max_acceleration>` if set. -->
+        <!-- DEPRECATED params from previous plugin implementation and therefore not set, could not find equivalent
+          max_wheel_acceleration 2.8
+          same as with update_rate 1000.0
+        -->
+        <topic>${prefix}cmd_vel</topic>
+        <odom_topic>${prefix}odom</odom_topic>
+        <frame_id>${prefix}odom</frame_id>
+        <child_frame_id>${prefix}base_footprint</child_frame_id>
+        <odom_publish_frequency>100</odom_publish_frequency>
+        <tf_topic>/tf</tf_topic>
       </plugin>
     </gazebo>
@@ -52,5 +86,8 @@
     <xacro:set_wheel_friction link="${prefix}br_caster_wheel_link" friction="1"/>
   </xacro:macro>
- <!-- See https://github.com/ros-simulation/gazebo_ros_pkgs/wiki/ROS-2-Migration:-P3D for ros2 information -->
+  <!-- Not yet migrated to ROS 2, and not sure why is needed, probably as ground truth for fake localization?
+    If we want to migrate it in future, perhaps see
+    https://github.com/ros-simulation/gazebo_ros_pkgs/wiki/ROS-2-Migration:-P3D for ros2 information
+    although I think is not gazebo harmonic compatible, so we would need to adapt it
   <xacro:macro name="p3d_base_controller" params="prefix">
     <gazebo>
@@ -68,4 +105,77 @@
       </plugin>
     </gazebo>
+  </xacro:macro> -->
+  <!-- imu plugin, see code under
+    https://github.com/gazebosim/gz-sim/blob/gz-sim8/src/systems/imu/Imu.hh
+    https://github.com/gazebosim/gz-sensors/blob/gz-sensors8/include/gz/sensors/ImuSensor.hh and documentation under
+    https://gazebosim.org/docs/harmonic/sensors/ -->
+  <xacro:macro name="imu_gazebo" params="prefix link stdev imu_topic update_rate">
+    <gazebo>
+      <plugin filename="gz-sim-imu-system" name="gz::sim::systems::Imu"/>
+    </gazebo>
+    <gazebo reference="${prefix}${link}">
+      <sensor name="imu_sensor" type="imu">
+        <pose relative_to="${prefix}${link}">0 0 0 0 0 0</pose>
+        <gz_frame_id>${prefix}${link}</gz_frame_id>
+        <update_rate>${update_rate}</update_rate>
+        <topic>${prefix}${imu_topic}</topic>
+        <always_on>1</always_on>
+        <visualize>true</visualize>
+        <imu>
+          <angular_velocity>
+            <x>
+              <noise type="gaussian">
+                <mean>0.0</mean>
+                <stddev>${stdev}</stddev>
+                <bias_mean>0.0000075</bias_mean>
+                <bias_stddev>0.0000008</bias_stddev>
+              </noise>
+            </x>
+            <y>
+              <noise type="gaussian">
+                <mean>0.0</mean>
+                <stddev>${stdev}</stddev>
+                <bias_mean>0.0000075</bias_mean>
+                <bias_stddev>0.0000008</bias_stddev>
+              </noise>
+            </y>
+            <z>
+              <noise type="gaussian">
+                <mean>0.0</mean>
+                <stddev>${stdev}</stddev>
+                <bias_mean>0.0000075</bias_mean>
+                <bias_stddev>0.0000008</bias_stddev>
+              </noise>
+            </z>
+          </angular_velocity>
+          <linear_acceleration>
+            <x>
+              <noise type="gaussian">
+                <mean>0.0</mean>
+                <stddev>${stdev}</stddev>
+                <bias_mean>0.1</bias_mean>
+                <bias_stddev>0.001</bias_stddev>
+              </noise>
+            </x>
+            <y>
+              <noise type="gaussian">
+                <mean>0.0</mean>
+                <stddev>${stdev}</stddev>
+                <bias_mean>0.1</bias_mean>
+                <bias_stddev>0.001</bias_stddev>
+              </noise>
+            </y>
+            <z>
+              <noise type="gaussian">
+                <mean>0.0</mean>
+                <stddev>${stdev}</stddev>
+                <bias_mean>0.1</bias_mean>
+                <bias_stddev>0.001</bias_stddev>
+              </noise>
+            </z>
+          </linear_acceleration>
+        </imu>
+      </sensor>
+    </gazebo>
   </xacro:macro>
 </robot>

File: mir_description/urdf/include/mir.transmission.xacro (robot description, xacro)
@@ -1,4 +1,4 @@
 <?xml version="1.0"?>
-<robot xmlns:xacro="http://ros.org/wiki/xacro">
+<robot xmlns:xacro="http://www.ros.org/wiki/xacro">
   <xacro:macro name="mir_wheel_transmission" params="prefix locationprefix">
     <transmission name="${prefix}${locationprefix}_wheel_trans">

File: mir_description/urdf/include/mir_v1.urdf.xacro (robot description, xacro)
@@ -1,8 +1,7 @@
 <?xml version="1.0"?>
-<robot xmlns:xacro="http://ros.org/wiki/xacro">
+<robot xmlns:xacro="http://www.ros.org/wiki/xacro">
   <xacro:arg name="mir_type" default="mir_100" />      <!-- The MiR variant. Can be "mir_100" or "mir_250" for now.-->
   <xacro:property name="mir_type" value="$(arg mir_type)" />  <!-- necessary because args cannot be accessed inside ${} expressions -->
   <xacro:include filename="$(find mir_description)/urdf/include/common_properties.urdf.xacro" />
-  <xacro:include filename="$(find mir_description)/urdf/include/imu.gazebo.urdf.xacro" />
   <xacro:include filename="$(find mir_description)/urdf/include/mir.gazebo.xacro" />
   <xacro:include filename="$(find mir_description)/urdf/include/mir.transmission.xacro" />
@@ -57,8 +56,12 @@
     </link>
     <gazebo reference="${prefix}${locationprefix}_wheel_link">
-      <material>Gazebo/FlatBlack</material>
+      <material>  <!-- Gazebo/FlatBlack -->
+        <ambient>0.1 0.1 0.1 1</ambient>
+        <diffuse>0.1 0.1 0.1 1</diffuse>
+        <specular>0.01 0.01 0.01 1</specular>
+      </material>
     </gazebo>
   </xacro:macro>
-  <xacro:macro name="caster_wheel" params="prefix ns locationprefix locationright wheel_base_dx">
+  <xacro:macro name="caster_wheel" params="prefix locationprefix locationright wheel_base_dx">
     <!-- caster hub -->
     <joint name="${prefix}${locationprefix}_caster_rotation_joint" type="continuous">
@@ -69,13 +72,4 @@
       <dynamics damping="0.01" friction="0.0"/>
     </joint>
-    <gazebo>
-      <plugin name="${locationprefix}_caster_rotation_joint_states" filename="libgazebo_ros_joint_state_publisher.so">
-        <ros>
-          <namespace>${ns}</namespace>
-        </ros>
-        <update_rate>200.0</update_rate>
-        <joint_name>${prefix}${locationprefix}_caster_rotation_joint</joint_name>
-      </plugin>
-    </gazebo>
     <link name="${prefix}${locationprefix}_caster_rotation_link">
       <inertial>
@@ -106,5 +100,9 @@
     </link>
     <gazebo reference="${prefix}${locationprefix}_caster_rotation_link">
-      <material>Gazebo/Grey</material>
+      <material> <!-- Gazebo/Grey-->
+        <ambient>0.3 0.3 0.3 1</ambient>
+        <diffuse>0.7 0.7 0.7 1</diffuse>
+        <specular>0.01 0.01 0.01 1</specular>
+      </material>
     </gazebo>
     <!-- caster wheel -->
@@ -115,13 +113,4 @@
       <axis xyz="0 1 0" />
     </joint>
-    <gazebo>
-      <plugin name="${locationprefix}_caster_wheel_joint_states" filename="libgazebo_ros_joint_state_publisher.so">
-        <ros>
-          <namespace>${ns}</namespace>
-        </ros>
-        <update_rate>200.0</update_rate>
-        <joint_name>${prefix}${locationprefix}_caster_wheel_joint</joint_name>
-      </plugin>
-    </gazebo>
     <link name="${prefix}${locationprefix}_caster_wheel_link">
       <xacro:cylinder_inertial mass="${mir_caster_wheel_mass}" radius="${mir_caster_wheel_radius}" length="${mir_caster_wheel_width}">
@@ -143,8 +132,12 @@
     </link>
     <gazebo reference="${prefix}${locationprefix}_caster_wheel_link">
-      <material>Gazebo/FlatBlack</material>
+      <material> <!-- Gazebo/FlatBlack -->
+        <ambient>0.1 0.1 0.1 1</ambient>
+        <diffuse>0.1 0.1 0.1 1</diffuse>
+        <specular>0.01 0.01 0.01 1</specular>
+      </material>
     </gazebo>
   </xacro:macro>
-  <xacro:macro name="mir" params="prefix ns">
+  <xacro:macro name="mir" params="prefix">
     <link name="${prefix}base_footprint" />
     <joint name="${prefix}base_joint" type="fixed">
@@ -172,5 +165,9 @@
     </link>
     <gazebo reference="${prefix}base_link">
-      <material>Gazebo/White</material>
+      <material> <!-- Gazebo/White -->
+        <ambient>1 1 1 1</ambient>
+        <diffuse>1 1 1 1</diffuse>
+        <specular>0.1 0.1 0.1 1</specular>
+      </material>
     </gazebo>
     <!-- IMU -->
@@ -181,5 +178,4 @@
     </joint>
     <link name="${prefix}imu_link" />
-    <xacro:imu_gazebo link="${prefix}imu_link" imu_topic="${prefix}imu_data" update_rate="50.0" stdev="${imu_stdev}" />
     <!-- Create an alias for imu_link. This is necessary because the real MiR's
          TF has imu_link, but the imu_data topic is published in the imu_frame
@@ -228,8 +224,8 @@
     <xacro:actuated_wheel prefix="${prefix}" locationprefix="left" locationright="-1"/>
     <xacro:actuated_wheel prefix="${prefix}" locationprefix="right" locationright="1"/>
-    <xacro:caster_wheel prefix="${prefix}" ns="${ns}" locationprefix="fl" locationright="-1" wheel_base_dx="${mir_front_caster_wheel_base_dx + mir_act_wheel_dx}"/>
-    <xacro:caster_wheel prefix="${prefix}" ns="${ns}" locationprefix="fr" locationright="1" wheel_base_dx="${mir_front_caster_wheel_base_dx + mir_act_wheel_dx}"/>
-    <xacro:caster_wheel prefix="${prefix}" ns="${ns}" locationprefix="bl" locationright="-1" wheel_base_dx="${-mir_back_caster_wheel_base_dx + mir_act_wheel_dx}"/>
-    <xacro:caster_wheel prefix="${prefix}" ns="${ns}" locationprefix="br" locationright="1" wheel_base_dx="${-mir_back_caster_wheel_base_dx + mir_act_wheel_dx}"/>
+    <xacro:caster_wheel prefix="${prefix}" locationprefix="fl" locationright="-1" wheel_base_dx="${mir_front_caster_wheel_base_dx + mir_act_wheel_dx}"/>
+    <xacro:caster_wheel prefix="${prefix}" locationprefix="fr" locationright="1" wheel_base_dx="${mir_front_caster_wheel_base_dx + mir_act_wheel_dx}"/>
+    <xacro:caster_wheel prefix="${prefix}" locationprefix="bl" locationright="-1" wheel_base_dx="${-mir_back_caster_wheel_base_dx + mir_act_wheel_dx}"/>
+    <xacro:caster_wheel prefix="${prefix}" locationprefix="br" locationright="1" wheel_base_dx="${-mir_back_caster_wheel_base_dx + mir_act_wheel_dx}"/>
     <joint name="${prefix}base_link_surface_joint" type="fixed">
       <origin xyz="${mir_act_wheel_dx} 0 0.352" rpy="0 0 0" />
@@ -242,5 +238,25 @@
     <!-- set the gazebo friction parameters for the wheels -->
     <xacro:set_all_wheel_frictions prefix="${prefix}"/>
-    <xacro:p3d_base_controller prefix="${prefix}" />
+    <!-- Simulation -->
+    <!-- publish the joint state of the wheels in simulation -->
+    <xacro:joint_states_plugin_gazebo prefix="${prefix}"
+        topic="joint_states"
+        left_wheel_joint="left_wheel_joint"
+        right_wheel_joint="right_wheel_joint"/>
+    <!-- I think this was required to publish ground truth for fake localization but I am not sure. -->
+    <!-- <xacro:p3d_base_controller prefix="${prefix}" /> -->
+    <xacro:diff_controller_plugin_gazebo prefix="${prefix}"
+        left_wheel_joint="${prefix}left_wheel_joint"
+        right_wheel_joint="${prefix}right_wheel_joint"
+        wheel_separation="${2*mir_act_wheel_dy}"
+        wheel_radius="${mir_act_wheel_radius}"/>
+    <!-- Required by lidar in simulation -->
+    <xacro:sensors_system_plugin />
+    <!-- Simulated imu -->
+    <xacro:imu_gazebo prefix="${prefix}"
+        link="imu_link"
+        stdev="${imu_stdev}"
+        imu_topic="imu_data"
+        update_rate="50.0"/>
   </xacro:macro>
 </robot>

File: mir_description/urdf/include/sick_s300.urdf.xacro (robot description, xacro)
@@ -1,4 +1,4 @@
 <?xml version="1.0"?>
-<robot xmlns:xacro="http://ros.org/wiki/xacro">
+<robot xmlns:xacro="http://www.ros.org/wiki/xacro">
   <xacro:include filename="$(find mir_description)/urdf/include/common_properties.urdf.xacro" />
   <xacro:property name="laser_x" value="0.156" />
@@ -27,8 +27,12 @@
     </link>
     <gazebo reference="${prefix}${link}">
-      <!-- <material value="Gazebo/Yellow" /> -->
-      <material value="Gazebo/FlatBlack" />
-      <sensor type="ray" name="${prefix}${link}">
-        <visualize>false</visualize>
+      <material> <!-- Gazebo/FlatBlack -->
+        <ambient>0.1 0.1 0.1 1</ambient>
+        <diffuse>0.1 0.1 0.1 1</diffuse>
+        <specular>0.01 0.01 0.01 1</specular>
+      </material>
+      <sensor name="${prefix}${link}" type="gpu_lidar">
+        <pose relative_to="${prefix}${link}">0 0 0 0 0 0</pose>
+        <topic>${prefix}${topic}</topic>
         <update_rate>12.5</update_rate>
         <ray>
@@ -40,4 +44,10 @@
               <max_angle>2.35619449615</max_angle>
             </horizontal>
+            <vertical>
+                <samples>1</samples>
+                <resolution>0.01</resolution>
+                <min_angle>0</min_angle>
+                <max_angle>0</max_angle>
+            </vertical>
           </scan>
           <range>
@@ -55,11 +65,7 @@
           </noise>
         </ray>
-        <plugin name="gazebo_ros_${link}_controller" filename="libgazebo_ros_ray_sensor.so">
-          <ros>
-            <remapping>~/out:=${prefix}${topic}</remapping>
-          </ros>
-          <output_type>sensor_msgs/LaserScan</output_type>
-          <frame_name>${prefix}${link}</frame_name>
-        </plugin>
+        <always_on>1</always_on>
+        <visualize>false</visualize>
+        <gz_frame_id>${prefix}${link}</gz_frame_id>
       </sensor>
     </gazebo>

File: mir_description/urdf/mir.urdf.xacro (robot description, xacro)
@@ -1,23 +1,15 @@
 <?xml version="1.0"?>
-<robot xmlns:xacro="http://ros.org/wiki/xacro"
-       name="mir" >
+<robot xmlns:xacro="http://www.ros.org/wiki/xacro"
+       name="mir_robot" >
   <!-- MiR base -->
   <xacro:include filename="$(find mir_description)/urdf/include/mir_v1.urdf.xacro" />
-  <xacro:include filename="$(find mir_description)/urdf/include/common.gazebo.xacro" />
-  <xacro:include filename="$(find mir_description)/urdf/include/mir.gazebo.xacro" />
   <xacro:arg name="tf_prefix" default="" />
-  <!-- prefix can not start with a slash like a global namespace! results in TF errors -->
-  <xacro:property name="ns" value="$(arg tf_prefix)" />
-  <xacro:if value="${ns == ''}">
+  <xacro:property name="tf_prefix_" value="$(arg tf_prefix)" />
+  <xacro:if value="${tf_prefix_ == ''}">
     <xacro:property name="prefix" value="" />
   </xacro:if>
-  <xacro:unless value="${ns == ''}">
-    <xacro:property name="prefix" value="${ns}/" />
+  <xacro:unless value="${tf_prefix_ == ''}">
+    <xacro:property name="prefix" value="${tf_prefix_}/" />
   </xacro:unless>
-  <xacro:mir prefix="${prefix}" ns="${ns}"/>
-  <xacro:diff_controller_plugin_gazebo prefix="${prefix}" ns="${ns}"
-    left_wheel_joint="${prefix}left_wheel_joint"
-    right_wheel_joint="${prefix}right_wheel_joint"
-    wheel_separation="${2*mir_act_wheel_dy}"
-    wheel_radius="${mir_act_wheel_radius}"/>
+  <xacro:mir prefix="${prefix}"/>
 </robot>
