Commit message: Gazebo: rviz-only material tags now apply to models in Gazebo

File: mir_description/urdf/include/common_properties.urdf.xacro (robot description, xacro)
@@ -4,5 +4,5 @@
  -->
 <robot name="xacro_properties" xmlns:xacro="http://www.ros.org/wiki/xacro">
-  <!-- #################### RViz materials #################### -->
+  <!-- #################### RViz and Gazebo materials #################### -->
   <xacro:property name="material_white">
     <material name="white">

File: mir_description/urdf/include/mir_v1.urdf.xacro (robot description, xacro)
@@ -55,11 +55,4 @@
       </collision>
     </link>
-    <gazebo reference="${prefix}${locationprefix}_wheel_link">
-      <material>  <!-- Gazebo/FlatBlack -->
-        <ambient>0.1 0.1 0.1 1</ambient>
-        <diffuse>0.1 0.1 0.1 1</diffuse>
-        <specular>0.01 0.01 0.01 1</specular>
-      </material>
-    </gazebo>
   </xacro:macro>
   <xacro:macro name="caster_wheel" params="prefix locationprefix locationright wheel_base_dx">
@@ -99,11 +92,4 @@
       </collision>
     </link>
-    <gazebo reference="${prefix}${locationprefix}_caster_rotation_link">
-      <material> <!-- Gazebo/Grey-->
-        <ambient>0.3 0.3 0.3 1</ambient>
-        <diffuse>0.7 0.7 0.7 1</diffuse>
-        <specular>0.01 0.01 0.01 1</specular>
-      </material>
-    </gazebo>
     <!-- caster wheel -->
     <joint name="${prefix}${locationprefix}_caster_wheel_joint" type="continuous">
@@ -131,11 +117,4 @@
       </collision>
     </link>
-    <gazebo reference="${prefix}${locationprefix}_caster_wheel_link">
-      <material> <!-- Gazebo/FlatBlack -->
-        <ambient>0.1 0.1 0.1 1</ambient>
-        <diffuse>0.1 0.1 0.1 1</diffuse>
-        <specular>0.01 0.01 0.01 1</specular>
-      </material>
-    </gazebo>
   </xacro:macro>
   <xacro:macro name="mir" params="prefix">
@@ -164,11 +143,4 @@
       </collision>
     </link>
-    <gazebo reference="${prefix}base_link">
-      <material> <!-- Gazebo/White -->
-        <ambient>1 1 1 1</ambient>
-        <diffuse>1 1 1 1</diffuse>
-        <specular>0.1 0.1 0.1 1</specular>
-      </material>
-    </gazebo>
     <!-- IMU -->
     <joint name="${prefix}base_link_to_imu_joint" type="fixed">

File: mir_description/urdf/include/sick_s300.urdf.xacro (robot description, xacro)
@@ -27,9 +27,4 @@
     </link>
     <gazebo reference="${prefix}${link}">
-      <material> <!-- Gazebo/FlatBlack -->
-        <ambient>0.1 0.1 0.1 1</ambient>
-        <diffuse>0.1 0.1 0.1 1</diffuse>
-        <specular>0.01 0.01 0.01 1</specular>
-      </material>
       <sensor name="${prefix}${link}" type="gpu_lidar">
         <pose relative_to="${prefix}${link}">0 0 0 0 0 0</pose>
